File: pcb/adcsd_shield.brd (EAGLE design)
At the start: 56.2 x 41.3 mm, 20 parts, among them X1 MCP3208

Commit message: some circuit modifications, updates
Parts:
- added C6: 1uF, rcl:C0402
- added IC2: MC1541TT, microchip:SOT23
- moved C2 4.96 mm to (57.1, 31.8), turned to 90 degrees
- moved C1 2.62 mm to (55.9, 31.8), turned to 90 degrees
- moved X1 2.54 mm to (50.2, 21.0)
- moved SL1 1.27 mm to (50.8, 35.6)
Connections:
- new net N$9: C6.1, IC2.2, X1.P$15
- net 5V: now also IC2.1; no longer X1.P$15
- net AGND: now also C6.2, IC2.3
Routing:
- net N$9: track 0.00 -> 4.16 mm
- net SPIN: track 34.5 -> 37.1 mm
- net DPIN: track 30.6 -> 33.1 mm
- net CPIN: track 24.4 -> 27.0 mm
- net 5V: track 67.4 -> 68.4 mm
- net CH3: track 15.9 -> 16.8 mm
- net CH2: track 12.3 -> 12.8 mm
- net CH1: track 8.67 -> 9.20 mm
- net CH0: track 4.71 -> 5.23 mm

Commit message: playing with simulation, updating component values accordingly
decreasing distortion
component values in the simulation are now more correct.
Parts:
- moved C5 1.27 mm to (77.5, 38.7)
Routing:
- net 3.3V: track 43.7 -> 42.4 mm
Changed lines of the file:
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@@
 <grid distance="0.025" unitdist="inch" unit="inch" style="lines" multiple="1" display="no" altdistance="0.025" altunitdist="inch" altunit="inch"/>
 <layers>
-<layer number="1" name="Top" color="4" fill="1" visible="no" active="yes"/>
+<layer number="1" name="Top" color="4" fill="1" visible="yes" active="yes"/>
 <layer number="16" name="Bottom" color="1" fill="1" visible="yes" active="yes"/>
 <layer number="17" name="Pads" color="2" fill="1" visible="yes" active="yes"/>
@@
 <element name="C1" library="rcl" package="C0402" value="0.1uF" x="55.88" y="31.75" rot="MR90"/>
 <element name="C2" library="rcl" package="C0402" value="1uF" x="57.15" y="31.75" rot="MR90"/>
-<element name="C5" library="rcl" package="C0402" value="1uF" x="78.74" y="38.735" rot="MR180"/>
+<element name="C5" library="rcl" package="C0402" value="1uF" x="77.47" y="38.735" rot="MR180"/>
 <element name="SL1" library="con-lsta" package="FE05-1" value="" x="50.8" y="35.56" rot="R180">
 <attribute name="OC_NEWARK" value="unknown" x="50.8" y="35.56" size="1.778" layer="27" rot="R180" display="off"/>
@@
 <via x="75.565" y="39.37" extent="1-16" drill="0.6"/>
 <wire x1="75.565" y1="39.37" x2="75.565" y2="41.06" width="0.4064" layer="16"/>
-<wire x1="78.09" y1="38.735" x2="76.2" y2="38.735" width="0.4064" layer="16"/>
+<wire x1="76.82" y1="38.735" x2="76.2" y2="38.735" width="0.4064" layer="16"/>
 <wire x1="76.2" y1="38.735" x2="75.565" y2="39.37" width="0.4064" layer="16"/>
 <wire x1="89.535" y1="41.275" x2="87.21" y2="41.275" width="0.6096" layer="16"/>
