File: pcb/preamp.brd (EAGLE design)
At the start: 59.4 x 43.2 mm, 50 parts, among them U1 LT1097CN8PBF, U2 LT1097CN8PBF, U3 LT1079CNPBF, U4 LT1079CNPBF

Commit message: some circuit modifications, updates
Parts:
- R1, R3: value 470 -> 3.3k
- R2, R4: value 3.3k -> 470
Changed lines of the file:
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@@
 <?xml version="1.0" encoding="utf-8"?>
 <!DOCTYPE eagle SYSTEM "eagle.dtd">
-<eagle version="6.6.0">
+<eagle version="7.3.0">
 <drawing>
 <settings>
@@
 <pass name="Default">
 <param name="RoutingGrid" value="50mil"/>
+<param name="AutoGrid" value="1"/>
+<param name="Efforts" value="0"/>
+<param name="TopRouterVariant" value="1"/>
 <param name="tpViaShape" value="round"/>
 <param name="PrefDir.1" value="|"/>
@@
 <element name="C9" library="resistor" package="C025-025X050" value="10uF" x="41.91" y="8.89"/>
 <element name="C10" library="resistor" package="C025-025X050" value="100nF" x="54.61" y="19.05" rot="R180"/>
-<element name="R1" library="resistor" package="0204/5" value="470" x="53.34" y="15.24"/>
-<element name="R2" library="resistor" package="0204/5" value="3.3k" x="48.26" y="12.7" rot="R180"/>
-<element name="R3" library="resistor" package="0204/5" value="470" x="41.91" y="40.64"/>
-<element name="R4" library="resistor" package="0204/5" value="3.3k" x="46.99" y="38.1"/>
+<element name="R1" library="resistor" package="0204/5" value="3.3k" x="53.34" y="15.24"/>
+<element name="R2" library="resistor" package="0204/5" value="470" x="48.26" y="12.7" rot="R180"/>
+<element name="R3" library="resistor" package="0204/5" value="3.3k" x="41.91" y="40.64"/>
+<element name="R4" library="resistor" package="0204/5" value="470" x="46.99" y="38.1"/>
 <element name="R8" library="resistor" package="0204/5" value="1.6k" x="20.32" y="43.18"/>
 <element name="R9" library="resistor" package="0204/5" value="16.2k" x="30.48" y="43.18"/>

Commit message: playing with simulation, updating component values accordingly
decreasing distortion
component values in the simulation are now more correct.
Parts:
- R18, R8: value 1.6k -> 22k
Changed lines of the file:
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@@
 <element name="R3" library="resistor" package="0204/5" value="3.3k" x="41.91" y="40.64"/>
 <element name="R4" library="resistor" package="0204/5" value="470" x="46.99" y="38.1"/>
-<element name="R8" library="resistor" package="0204/5" value="1.6k" x="20.32" y="43.18"/>
+<element name="R8" library="resistor" package="0204/5" value="22k" x="20.32" y="43.18"/>
 <element name="R9" library="resistor" package="0204/5" value="16.2k" x="30.48" y="43.18"/>
 <element name="R10" library="resistor" package="0204/5" value="7.9k" x="25.4" y="40.64" rot="R90"/>
@@
 <element name="R17" library="resistor" package="0204/7" value="220" x="7.62" y="10.16"/>
 <element name="C6" library="resistor" package="C050-030X075" value="10uF" x="20.32" y="10.16"/>
-<element name="R18" library="resistor" package="0204/5" value="1.6k" x="20.32" y="7.62"/>
+<element name="R18" library="resistor" package="0204/5" value="22k" x="20.32" y="7.62"/>
 <element name="R19" library="resistor" package="0204/5" value="7.9k" x="25.4" y="10.16" rot="R270"/>
 <element name="C11" library="resistor" package="C050-024X044" value=".015uF" x="33.02" y="10.16" rot="R180"/>

Commit message: updating schematic to reflect new component values
Parts:
- C11, C4: value .015uF -> 100nF
- C12: value 3300pF -> 10nF
- C5: value 3300pF -> 10n
- R10, R19: value 7.9k -> 1.19k
- R20, R9: value 16.2k -> 21.5k
Changed lines of the file:
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@@
 <element name="R4" library="resistor" package="0204/5" value="470" x="46.99" y="38.1"/>
 <element name="R8" library="resistor" package="0204/5" value="22k" x="20.32" y="43.18"/>
-<element name="R9" library="resistor" package="0204/5" value="16.2k" x="30.48" y="43.18"/>
-<element name="R10" library="resistor" package="0204/5" value="7.9k" x="25.4" y="40.64" rot="R90"/>
+<element name="R9" library="resistor" package="0204/5" value="21.5k" x="30.48" y="43.18"/>
+<element name="R10" library="resistor" package="0204/5" value="1.19k" x="25.4" y="40.64" rot="R90"/>
 <element name="R5" library="resistor" package="0204/7" value="560k" x="3.81" y="33.02" rot="R90"/>
 <element name="R6" library="resistor" package="0204/7" value="560k" x="6.35" y="39.37" rot="R270"/>
 <element name="R7" library="resistor" package="0204/7" value="220" x="8.89" y="39.37" rot="R270"/>
 <element name="C3" library="resistor" package="C050-030X075" value="10uF" x="20.32" y="39.37"/>
-<element name="C4" library="resistor" package="C050-024X044" value=".015uF" x="33.02" y="40.64" rot="R180"/>
-<element name="C5" library="resistor" package="C025-024X044" value="3300pF" x="36.83" y="43.18"/>
+<element name="C4" library="resistor" package="C050-024X044" value="100nF" x="33.02" y="40.64" rot="R180"/>
+<element name="C5" library="resistor" package="C025-024X044" value="10n" x="36.83" y="43.18"/>
 <element name="R11" library="resistor" package="0204/5" value="2k" x="43.18" y="34.29" rot="R270"/>
 <element name="R12" library="resistor" package="0204/5" value="500" x="44.45" y="29.21" rot="R270"/>
@@
 <element name="C6" library="resistor" package="C050-030X075" value="10uF" x="20.32" y="10.16"/>
 <element name="R18" library="resistor" package="0204/5" value="22k" x="20.32" y="7.62"/>
-<element name="R19" library="resistor" package="0204/5" value="7.9k" x="25.4" y="10.16" rot="R270"/>
-<element name="C11" library="resistor" package="C050-024X044" value=".015uF" x="33.02" y="10.16" rot="R180"/>
-<element name="R20" library="resistor" package="0204/5" value="16.2k" x="30.48" y="7.62"/>
-<element name="C12" library="resistor" package="C025-024X044" value="3300pF" x="36.83" y="7.62"/>
+<element name="R19" library="resistor" package="0204/5" value="1.19k" x="25.4" y="10.16" rot="R270"/>
+<element name="C11" library="resistor" package="C050-024X044" value="100nF" x="33.02" y="10.16" rot="R180"/>
+<element name="R20" library="resistor" package="0204/5" value="21.5k" x="30.48" y="7.62"/>
+<element name="C12" library="resistor" package="C025-024X044" value="10nF" x="36.83" y="7.62"/>
 <element name="R21" library="resistor" package="0204/5" value="2k" x="43.18" y="13.97" rot="R90"/>
 <element name="R22" library="resistor" package="0204/5" value="500" x="44.45" y="19.05" rot="R90"/>
